File: wss.kicad_sch (KiCad schematic)
At the start: 20 parts, among them J1 Conn_01x02, J2 Conn_01x02, J3 Conn_01x03, U2 TLV9061xDBV

Commit message: added schmitt trigger comparator
Parts:
- added U1: 74HC14, Package_DIP:DIP-14_W7.62mm, symbol 74xx:74HC14
- added V1: VSIN, symbol Simulation_SPICE:VSIN
- R8: value 560k -> 5.6M
Connections:
- net +3V3: now also U1.14 (VCC)
- net GND: now also U1.10, U1.11, U1.12, U1.13, U1.3, U1.4, U1.5, U1.6, U1.7 (GND), U1.8, U1.9, V1.2
- net Signal2: now also V1.1
- net Signal_Output: now also U1.2; no longer R9.2, U2.1
- new net: R9.2, U1.1, U2.1
